Commit message: created gazebo move control

File: description/robot.urdf.xacro (robot description, xacro)
@@ -3,3 +3,4 @@
     <!-- :include 把file放進來 -->
     <xacro:include filename="robot_core.xacro" />
+    <xacro:include filename="gazebo_control.xacro" />
 </robot>

File: description/robot_core.xacro (robot description, xacro)
@@ -27,4 +27,6 @@
     [set inertia] 利用那個已經有的包就好
     <xacro:include filename="inertial_macros.xacro"/>
+    [[Add Gazebo Tag]]輸進去gazebo之後, 會有一些問題, 所以要加上gazebo tag
+    1. 顏色消失 ==> 在每個有visual tag的"link包下面"都加上gazebo tag（把顏色對上gazebo內的顏色)
     -->
     <!-- set baselink(1st link for mobile robot) -->
@@ -60,4 +62,8 @@
         </xacro:inertial_box>
     </link>
+    <!-- [[Add Gazebo Tag]]1. 顏色消失 ==> 在每個有visual tag的"link包下面"都加上gazebo tag（把顏色對上gazebo內的顏色)-->
+    <gazebo reference="chassis">
+        <material>Gazebo/White</material>
+    </gazebo>
     <!-- Left wheel link -->
     <joint name="left_wheel_joint" type="continuous"><!-- 因為車車輪子會contunuously轉 -->
@@ -84,5 +90,8 @@
         </xacro:inertial_cylinder>
     </link>
-        <!-- Right wheel link -->
+    <gazebo reference="left_wheel">
+        <material>Gazebo/Blue</material>
+    </gazebo>
+    <!-- Right wheel link -->
     <joint name="right_wheel_joint" type="continuous"><!-- 因為車車輪子會contunuously轉 -->
         <parent link="base_link"/>
@@ -108,4 +117,7 @@
         </xacro:inertial_cylinder>
     </link>
+    <gazebo reference="right_wheel">
+        <material>Gazebo/Blue</material>
+    </gazebo>
     <!-- caster wheel link(有點像萬象輪的前輪,利用把它變成frictionless 所以可以不影響轉向來達成) -->
     <joint name="caster_wheel_joint" type="fixed">
@@ -131,3 +143,8 @@
         </xacro:inertial_sphere>
     </link>
+    <gazebo reference="caster_wheel"> <!-- 這項gazebo特徵是要加給caster_wheel這個"link"的 -->
+        <material>Gazebo/Black</material>
+        <mu1 value="0.001"/><!-- 因為想要這個萬象輪試frictionless所以設一個很小的數字, 也可以是0. 如果沒設成frictionless, 就會一直產生摩擦力導致車體bounce -->
+        <mu2 value="0.001"/><!-- 兩種小小不同的friction coeffition -->
+    </gazebo>
 </robot>
